File: SaLAltimeter.brd (EAGLE design)
At the start: 74.6 x 19.7 mm, 91 parts, among them U1 ATSAMD21G-A, U2 V_REG_LDOSMD, U3 ADXL345, Y3 32MHz

Commit message: finshed wiring
Parts:
- added R18: 100k, SparkFun-Passives:0402-RES
- added R19: 27k, SparkFun-Passives:0402-RES
- added R20: 10k, SparkFun-Passives:0402-RES
- C8: value (none) -> 0.1uF
- J1: value (none) -> BAT
- JP2: value (none) -> MAIN
- JP3: value (none) -> DROGUE
- R1, R13, R2, R3, R4: value (none) -> 10k
- R15: value (none) -> 18
- U4: value (none) -> gps
- Y1: value (none) -> 32.768kHx
- moved F1 10.6 mm to (48.3, 17.3), turned to 0 degrees
- moved R2 3.20 mm to (45.1, 1.65), turned to 0 degrees
- moved J$1 2.22 mm to (66.0, 2.67)
- moved R13 2.11 mm to (53.2, 3.68), turned to 270 degrees
- moved R4 2.01 mm to (33.0, 10.2), turned to 90 degrees
- moved STANDOFF1 1.97 mm to (65.4, 17.0)
- moved L4 1.94 mm to (62.5, 5.33)
- moved C10 1.94 mm to (32.1, 5.46), turned to 270 degrees
- moved R3 1.80 mm to (31.0, 3.17), turned to 90 degrees
- moved C39 1.61 mm to (25.9, 2.54), turned to 0 degrees
- moved JP4 1.52 mm to (57.5, 17.1)
- moved U$4 1.17 mm to (41.8, 5.33)
- moved L3 0.92 mm to (60.5, 5.46), turned to 270 degrees
- moved S2 0.90 mm to (49.8, 2.03)
- moved C32 0.89 mm to (43.2, 9.78)
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Connections:
- removed net N$7: U1.6
- net BUZZER: now also SG1.+, U1.21; no longer SG1.-, U1.27
- net CS_ACCEL: now also U1.25; no longer U1.24
- net CS_BARO: now also U1.14; no longer U1.22
- net CS_MEM: now also U1.13; no longer U1.23
- net CS_TX: now also R20.1, U1.15; no longer U1.28
- net FIRE_A: now also U1.47; no longer U1.45
- net FIRE_B: now also U1.48; no longer U1.46
- net GND: now also R19.1, R20.2, SG1.-, U$7.EXP, U$7.EXP@1, U$7.EXP@2, U$7.EXP@3, U$7.EXP@4, U$7.EXP@5, U$7.EXP@6, U$7.EXP@7, U$7.EXP@8, U$7.EXP@9; no longer SG1.+
- net LVD_IN: now also F1.2
- net N$5: now also U1.6
- net PROG: now also U1.12; no longer U1.29
- net RAW: now also R18.2
- net SENSE_BAT: now also R18.1, R19.2, U1.11; no longer U1.9
- net SPI_MISO: now also U1.23; no longer U1.21, U1.25
- net SPI_MOSI: now also U1.22; no longer U1.19, U1.26
- net SPI_SCK: now also U1.24; no longer U1.20
- net SWCLK: now also U1.45
- net SWDIO: now also U1.46
Routing:
- net GND: track 121.0 -> 383.4 mm, vias 23 -> 57
- net 3.3V: track 81.4 -> 232.9 mm, vias 9 -> 26
- net LVD_IN: track 36.8 -> 101.6 mm, vias 4 -> 6
- net USB_D+: track 0.00 -> 33.1 mm, vias 0 -> 1
- net SPI_MOSI: track 0.00 -> 32.8 mm, vias 0 -> 2
- net PROG: track 0.00 -> 31.3 mm, vias 0 -> 1
- net SPI_MISO: track 0.00 -> 30.8 mm, vias 0 -> 2
- net USB_D-: track 0.00 -> 30.6 mm, vias 0 -> 1
- net CS_TX: track 0.00 -> 27.2 mm, vias 0 -> 3
- net SPI_SCK: track 0.00 -> 25.8 mm, vias 0 -> 4
- net SWDIO: track 0.00 -> 21.2 mm, vias 0 -> 1
- net CS_MEM: track 0.00 -> 20.5 mm
- net SWCLK: track 0.00 -> 17.9 mm, vias 0 -> 1
- net SENSE_BAT: track 0.00 -> 14.0 mm
- net N$5: track 1.68 -> 14.2 mm, vias 0 -> 2
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- added copper zone on layer 15, net 3.3V
- added copper zone on layer 1, net GND
- added copper zone on layer 16, net GND
- added copper zone on layer 2, net GND
Other:
- board size 74.6 x 19.7 mm -> 73.3 x 19.7 mm

Commit message: mk1 finished!
Parts:
- removed U$7: CC1120, SaL-lib:CC1120
- added 1U2: V_REG_LDOSMD, SparkFun-PowerIC:SOT23-5
- U2: value V_REG_LDOSMD -> CC1120; device SparkFun-PowerIC:SOT23-5 -> SaL-lib:CC1120
- moved U2 33.5 mm to (48.3, 10.2), turned to 0 degrees
- moved JP2 2.79 mm to (9.65, 14.9), flipped to the bottom
- moved U$2 1.92 mm to (3.43, 16.5)
- moved F1 0.64 mm to (48.9, 17.3)
- moved STANDOFF1 0.25 mm to (65.4, 16.8)
- moved L6 0.13 mm to (57.9, 9.40)
- renumbered U$4 to MEM
Connections:
- net 3.3V: now also 1U2.5, U2.1, U2.12, U2.13, U2.15, U2.22, U2.27, U2.28; no longer U$7.1, U$7.12, U$7.13, U$7.15, U$7.22, U$7.27, U$7.28, U$7.5
- net CS_TX: now also U2.11; no longer U$7.11
- net FET_A: now also JP2.P2; no longer JP2.P1
- net GND: now also 1U2.2, U2.EXP, U2.EXP@1, U2.EXP@2, U2.EXP@3, U2.EXP@4, U2.EXP@5, U2.EXP@6, U2.EXP@7, U2.EXP@8, U2.EXP@9; no longer U$7.EXP, U$7.EXP@1, U$7.EXP@2, U$7.EXP@3, U$7.EXP@4, U$7.EXP@5, U$7.EXP@6, U$7.EXP@7, U$7.EXP@8, U$7.EXP@9, U2.2
- net LVD_IN: now also 1U2.1, 1U2.3, JP2.P1; no longer JP2.P2, U2.1, U2.3
- net N$15: now also U2.25; no longer U$7.25
- net N$16: now also U2.18; no longer U$7.18
- net N$17: now also U2.19; no longer U$7.19
- net N$19: now also U2.20; no longer U$7.20
- net N$20: now also U2.24; no longer U$7.24
- net N$21: now also U2.23; no longer U$7.23
- net N$22: now also U2.21; no longer U$7.21
- net N$23: now also U2.26; no longer U$7.26
- net N$24: now also U2.14; no longer U$7.14
- net N$25: now also U2.32; no longer U$7.32
- net N$26: now also U2.29; no longer U$7.29
- net N$27: now also U2.30; no longer U$7.30
- net N$28: now also U2.31; no longer U$7.31
- net N$34: now also U2.6; no longer U$7.6
- net N$9: now also U2.17; no longer U$7.17
- net SPI_MISO: now also U2.9; no longer U$7.9
- net SPI_MOSI: now also U2.7; no longer U$7.7
- net SPI_SCK: now also U2.8; no longer U$7.8
Routing:
- net GND: track 383.4 -> 388.3 mm
- net RAW: track 43.9 -> 45.8 mm
- net N$2: track 25.5 -> 27.3 mm

Commit message: parts lists added
Parts:
- C1: value 1.0uF -> 2.2uF
- R10, R12: value 10kohm -> 27K
- R11, R9: value 10kohm -> 100K
- R5, R8: value 10kohm -> 3.3k
- R6, R7: value 10kohm -> 100
Changed lines of the file:
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@@
 <attribute name="NAME" x="14.859" y="15.875" size="0.6096" layer="25" rot="R270"/>
 </element>
-<element name="C1" library="SparkFun-Capacitors" package="0603-CAP" value="1.0uF" x="15.875" y="12.573" smashed="yes">
+<element name="C1" library="SparkFun-Capacitors" package="0603-CAP" value="2.2uF" x="15.875" y="12.573" smashed="yes">
 <attribute name="NAME" x="17.399" y="12.446" size="0.4064" layer="25" font="vector"/>
 </element>
@@
 <attribute name="NAME" x="27.051" y="2.0955" size="0.6096" layer="25"/>
 </element>
-<element name="R5" library="SparkFun-Resistors" package="0402-RES" value="10kohm" x="13.081" y="11.43" smashed="yes">
+<element name="R5" library="SparkFun-Resistors" package="0402-RES" value="3.3k" x="13.081" y="11.43" smashed="yes">
 <attribute name="NAME" x="14.224" y="11.2395" size="0.6096" layer="25"/>
 </element>
-<element name="R6" library="SparkFun-Resistors" package="0402-RES" value="10kohm" x="13.081" y="10.033" smashed="yes" rot="R180">
+<element name="R6" library="SparkFun-Resistors" package="0402-RES" value="100" x="13.081" y="10.033" smashed="yes" rot="R180">
 <attribute name="NAME" x="14.224" y="9.7155" size="0.6096" layer="25"/>
 </element>
-<element name="R9" library="SparkFun-Resistors" package="0402-RES" value="10kohm" x="9.525" y="16.383" smashed="yes" rot="R180">
+<element name="R9" library="SparkFun-Resistors" package="0402-RES" value="100K" x="9.525" y="16.383" smashed="yes" rot="R180">
 <attribute name="NAME" x="8.382" y="16.7005" size="0.6096" layer="25" rot="R180"/>
 </element>
-<element name="R10" library="SparkFun-Resistors" package="0402-RES" value="10kohm" x="9.779" y="17.907" smashed="yes" rot="R180">
+<element name="R10" library="SparkFun-Resistors" package="0402-RES" value="27K" x="9.779" y="17.907" smashed="yes" rot="R180">
 <attribute name="NAME" x="8.636" y="18.0975" size="0.6096" layer="25" rot="R180"/>
 </element>
-<element name="R7" library="SparkFun-Resistors" package="0402-RES" value="10kohm" x="13.081" y="8.636" smashed="yes">
+<element name="R7" library="SparkFun-Resistors" package="0402-RES" value="100" x="13.081" y="8.636" smashed="yes">
 <attribute name="NAME" x="14.224" y="8.3185" size="0.6096" layer="25"/>
 </element>
-<element name="R8" library="SparkFun-Resistors" package="0402-RES" value="10kohm" x="13.081" y="7.239" smashed="yes" rot="R180">
+<element name="R8" library="SparkFun-Resistors" package="0402-RES" value="3.3k" x="13.081" y="7.239" smashed="yes" rot="R180">
 <attribute name="NAME" x="14.224" y="6.9215" size="0.6096" layer="25"/>
 </element>
-<element name="R11" library="SparkFun-Resistors" package="0402-RES" value="10kohm" x="9.525" y="3.175" smashed="yes">
+<element name="R11" library="SparkFun-Resistors" package="0402-RES" value="100K" x="9.525" y="3.175" smashed="yes">
 <attribute name="NAME" x="8.509" y="3.4925" size="0.6096" layer="25" rot="R180"/>
 </element>
-<element name="R12" library="SparkFun-Resistors" package="0402-RES" value="10kohm" x="9.525" y="1.778" smashed="yes" rot="R180">
+<element name="R12" library="SparkFun-Resistors" package="0402-RES" value="27K" x="9.525" y="1.778" smashed="yes" rot="R180">
 <attribute name="NAME" x="8.382" y="2.0955" size="0.6096" layer="25" rot="R180"/>
 </element>
