File: SaLAltimeter.sch (EAGLE design)
At the start: 87 parts, among them U1 ATSAMD21G-A, U2 V_REG_LDOSMD, U3 ADXL345, Y3 32MHz

Commit message: aligned tx parts
Connections:
- removed net MISO: U$4.SO, U$5.SDO, U$7.GPOI1, U3.SDO
- removed net MOSI: U$4.SI, U$5.SDI/SDA, U$7.SI, U3.SDA
- removed net RX_GPS: U4.TX
- removed net SCK: U$4.SCK, U$5.SCLK, U$7.SCLK, U3.SCL
- removed net TX_GPS: U4.RX
- new net GPS_RX: U1.PA11(AIN19/SER0:3+), U4.TX
- new net GPS_TX: U1.PA10(AIN18/SER0:2+), U4.RX
- new net SPI_MISO: U$4.SO, U$5.SDO, U$7.GPOI1, U1.PA12(I2C/SER2:0+), U3.SDO
- new net SPI_MOSI: U$4.SI, U$5.SDI/SDA, U$7.SI, U1.PB10(SER4:2+), U3.SDA
- new net SPI_SCK: U$4.SCK, U$5.SCLK, U$7.SCLK, U1.PB11(SER4:3+), U3.SCL
- net CS_ACCEL: now also U1.PA15(XOUT/SER2:3+)
- net CS_BARO: now also U1.PA13(I2C/SER2:1+)
- net CS_MEM: now also U1.PA14(XIN/SER2:2+)
- net CS_TX: now also U1.PA16(I2C/SER1:0+)
- net PROG: now also U1.PA17(I2C/SER1:1+)
Changed lines of the file:
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@@
 <label x="40.64" y="116.84" size="1.27" layer="95" xref="yes"/>
 </segment>
-</net>
-<net name="SCK" class="0">
-<segment>
-<pinref part="U$4" gate="G$1" pin="SCK"/>
-<wire x1="35.56" y1="114.3" x2="38.1" y2="114.3" width="0.1524" layer="91"/>
-<label x="38.1" y="114.3" size="1.27" layer="97" xref="yes"/>
-</segment>
-<segment>
-<pinref part="U$5" gate="G$1" pin="SCLK"/>
-<wire x1="38.1" y1="78.74" x2="40.64" y2="78.74" width="0.1524" layer="91"/>
-<label x="40.64" y="78.74" size="1.27" layer="95" xref="yes"/>
-</segment>
-<segment>
-<pinref part="U3" gate="G$1" pin="SCL"/>
-<wire x1="40.64" y1="35.56" x2="43.18" y2="35.56" width="0.1524" layer="91"/>
-<label x="43.18" y="35.56" size="1.27" layer="95" xref="yes"/>
-</segment>
-<segment>
-<pinref part="U$7" gate="G$1" pin="SCLK"/>
-<wire x1="309.88" y1="208.28" x2="309.88" y2="195.58" width="0.1524" layer="91"/>
-<wire x1="309.88" y1="195.58" x2="304.8" y2="195.58" width="0.1524" layer="91"/>
-<label x="304.8" y="195.58" size="1.27" layer="95" rot="R180" xref="yes"/>
-</segment>
-</net>
-<net name="MOSI" class="0">
-<segment>
-<pinref part="U$4" gate="G$1" pin="SI"/>
-<wire x1="35.56" y1="111.76" x2="38.1" y2="111.76" width="0.1524" layer="91"/>
-<label x="38.1" y="111.76" size="1.27" layer="95" xref="yes"/>
-</segment>
-<segment>
-<pinref part="U$5" gate="G$1" pin="SDI/SDA"/>
-<wire x1="38.1" y1="76.2" x2="40.64" y2="76.2" width="0.1524" layer="91"/>
-<label x="40.64" y="76.2" size="1.27" layer="95" xref="yes"/>
-</segment>
-<segment>
-<pinref part="U3" gate="G$1" pin="SDA"/>
-<wire x1="40.64" y1="38.1" x2="43.18" y2="38.1" width="0.1524" layer="91"/>
-<label x="43.18" y="38.1" size="1.27" layer="95" xref="yes"/>
-</segment>
-<segment>
-<pinref part="U$7" gate="G$1" pin="SI"/>
-<wire x1="309.88" y1="210.82" x2="307.34" y2="210.82" width="0.1524" layer="91"/>
-<wire x1="307.34" y1="210.82" x2="307.34" y2="198.12" width="0.1524" layer="91"/>
-<wire x1="307.34" y1="198.12" x2="304.8" y2="198.12" width="0.1524" layer="91"/>
-<label x="304.8" y="198.12" size="1.27" layer="95" rot="R180" xref="yes"/>
-</segment>
-</net>
-<net name="MISO" class="0">
-<segment>
-<pinref part="U$4" gate="G$1" pin="SO"/>
-<wire x1="35.56" y1="109.22" x2="38.1" y2="109.22" width="0.1524" layer="91"/>
-<label x="38.1" y="109.22" size="1.27" layer="95" xref="yes"/>
-</segment>
-<segment>
-<pinref part="U$5" gate="G$1" pin="SDO"/>
-<wire x1="38.1" y1="73.66" x2="40.64" y2="73.66" width="0.1524" layer="91"/>
-<label x="40.64" y="73.66" size="1.27" layer="95" xref="yes"/>
-</segment>
-<segment>
-<pinref part="U3" gate="G$1" pin="SDO"/>
-<wire x1="40.64" y1="40.64" x2="43.18" y2="40.64" width="0.1524" layer="91"/>
-<label x="43.18" y="40.64" size="1.27" layer="95" xref="yes"/>
-</segment>
-<segment>
-<pinref part="U$7" gate="G$1" pin="GPOI1"/>
-<wire x1="320.04" y1="195.58" x2="320.04" y2="193.04" width="0.1524" layer="91"/>
-<wire x1="320.04" y1="193.04" x2="304.8" y2="193.04" width="0.1524" layer="91"/>
-<label x="304.8" y="193.04" size="1.27" layer="95" rot="R180" xref="yes"/>
+<segment>
+<pinref part="U1" gate="G$1" pin="PA14(XIN/SER2:2+)"/>
+<wire x1="200.66" y1="193.04" x2="203.2" y2="193.04" width="0.1524" layer="91" style="longdash"/>
+<label x="203.2" y="193.04" size="1.27" layer="95" xref="yes"/>
 </segment>
 </net>
@@
 <label x="43.18" y="81.28" size="1.27" layer="95" xref="yes"/>
 </segment>
+<segment>
+<pinref part="U1" gate="G$1" pin="PA13(I2C/SER2:1+)"/>
+<wire x1="200.66" y1="195.58" x2="203.2" y2="195.58" width="0.1524" layer="91" style="longdash"/>
+<label x="203.2" y="195.58" size="1.27" layer="95" xref="yes"/>
+</segment>
 </net>
 <net name="CS_ACCEL" class="0">
@@
 <junction x="43.18" y="45.72"/>
 <label x="43.18" y="45.72" size="1.27" layer="95" xref="yes"/>
+</segment>
+<segment>
+<pinref part="U1" gate="G$1" pin="PA15(XOUT/SER2:3+)"/>
+<wire x1="200.66" y1="190.5" x2="203.2" y2="190.5" width="0.1524" layer="91" style="longdash"/>
+<label x="203.2" y="190.5" size="1.27" layer="95" xref="yes"/>
 </segment>
 </net>
@@
 <label x="15.24" y="157.48" size="1.27" layer="95" rot="R180" xref="yes"/>
 </segment>
+<segment>
+<pinref part="U1" gate="G$1" pin="PA17(I2C/SER1:1+)"/>
+<wire x1="200.66" y1="185.42" x2="203.2" y2="185.42" width="0.1524" layer="91" style="longdash"/>
+<label x="203.2" y="185.42" size="1.27" layer="95" xref="yes"/>
+</segment>
 </net>
 <net name="N$9" class="0">
@@
 <label x="304.8" y="190.5" size="1.27" layer="95" rot="R180" xref="yes"/>
 </segment>
+<segment>
+<pinref part="U1" gate="G$1" pin="PA16(I2C/SER1:0+)"/>
+<wire x1="200.66" y1="187.96" x2="203.2" y2="187.96" width="0.1524" layer="91" style="longdash"/>
+<label x="203.2" y="187.96" size="1.27" layer="95" xref="yes"/>
+</segment>
 </net>
 <net name="N$30" class="0">
@@
 </segment>
 </net>
-<net name="RX_GPS" class="0">
+<net name="GPS_RX" class="0">
 <segment>
 <pinref part="U4" gate="G$1" pin="TX"/>
@@
 <label x="337.82" y="88.9" size="1.27" layer="95" rot="R180" xref="yes"/>
 </segment>
-</net>
-<net name="TX_GPS" class="0">
+<segment>
+<pinref part="U1" gate="G$1" pin="PA11(AIN19/SER0:3+)"/>
+<wire x1="200.66" y1="200.66" x2="203.2" y2="200.66" width="0.1524" layer="91" style="longdash"/>
+<label x="203.2" y="200.66" size="1.27" layer="95" xref="yes"/>
+</segment>
+</net>
+<net name="SPI_MISO" class="0">
+<segment>
+<pinref part="U1" gate="G$1" pin="PA12(I2C/SER2:0+)"/>
+<wire x1="200.66" y1="198.12" x2="203.2" y2="198.12" width="0.1524" layer="91" style="longdash"/>
+<label x="203.2" y="198.12" size="1.27" layer="95" xref="yes"/>
+</segment>
+<segment>
+<pinref part="U$4" gate="G$1" pin="SO"/>
+<wire x1="35.56" y1="109.22" x2="38.1" y2="109.22" width="0.1524" layer="91"/>
+<label x="38.1" y="109.22" size="1.27" layer="95" xref="yes"/>
+</segment>
+<segment>
+<pinref part="U$5" gate="G$1" pin="SDO"/>
+<wire x1="38.1" y1="73.66" x2="40.64" y2="73.66" width="0.1524" layer="91"/>
+<label x="40.64" y="73.66" size="1.27" layer="95" xref="yes"/>
+</segment>
+<segment>
+<pinref part="U3" gate="G$1" pin="SDO"/>
+<wire x1="40.64" y1="40.64" x2="43.18" y2="40.64" width="0.1524" layer="91"/>
+<label x="43.18" y="40.64" size="1.27" layer="95" xref="yes"/>
+</segment>
+<segment>
+<pinref part="U$7" gate="G$1" pin="GPOI1"/>
+<wire x1="320.04" y1="195.58" x2="320.04" y2="193.04" width="0.1524" layer="91"/>
+<wire x1="320.04" y1="193.04" x2="304.8" y2="193.04" width="0.1524" layer="91"/>
+<label x="304.8" y="193.04" size="1.27" layer="95" rot="R180" xref="yes"/>
+</segment>
+</net>
+<net name="SPI_MOSI" class="0">
+<segment>
+<pinref part="U1" gate="G$1" pin="PB10(SER4:2+)"/>
+<wire x1="200.66" y1="149.86" x2="203.2" y2="149.86" width="0.1524" layer="91" style="longdash"/>
+<label x="203.2" y="149.86" size="1.27" layer="95" xref="yes"/>
+</segment>
+<segment>
+<pinref part="U$4" gate="G$1" pin="SI"/>
+<wire x1="35.56" y1="111.76" x2="38.1" y2="111.76" width="0.1524" layer="91"/>
+<label x="38.1" y="111.76" size="1.27" layer="95" xref="yes"/>
+</segment>
+<segment>
+<pinref part="U$5" gate="G$1" pin="SDI/SDA"/>
+<wire x1="38.1" y1="76.2" x2="40.64" y2="76.2" width="0.1524" layer="91"/>
+<label x="40.64" y="76.2" size="1.27" layer="95" xref="yes"/>
+</segment>
+<segment>
+<pinref part="U3" gate="G$1" pin="SDA"/>
+<wire x1="40.64" y1="38.1" x2="43.18" y2="38.1" width="0.1524" layer="91"/>
+<label x="43.18" y="38.1" size="1.27" layer="95" xref="yes"/>
+</segment>
+<segment>
+<pinref part="U$7" gate="G$1" pin="SI"/>
+<wire x1="309.88" y1="210.82" x2="307.34" y2="210.82" width="0.1524" layer="91"/>
+<wire x1="307.34" y1="210.82" x2="307.34" y2="198.12" width="0.1524" layer="91"/>
+<wire x1="307.34" y1="198.12" x2="304.8" y2="198.12" width="0.1524" layer="91"/>
+<label x="304.8" y="198.12" size="1.27" layer="95" rot="R180" xref="yes"/>
+</segment>
+</net>
+<net name="SPI_SCK" class="0">
+<segment>
+<pinref part="U1" gate="G$1" pin="PB11(SER4:3+)"/>
+<wire x1="200.66" y1="147.32" x2="203.2" y2="147.32" width="0.1524" layer="91" style="longdash"/>
+<label x="203.2" y="147.32" size="1.27" layer="95" xref="yes"/>
+</segment>
+<segment>
+<pinref part="U$4" gate="G$1" pin="SCK"/>
+<wire x1="35.56" y1="114.3" x2="38.1" y2="114.3" width="0.1524" layer="91"/>
+<label x="38.1" y="114.3" size="1.27" layer="97" xref="yes"/>
+</segment>
+<segment>
+<pinref part="U$5" gate="G$1" pin="SCLK"/>
+<wire x1="38.1" y1="78.74" x2="40.64" y2="78.74" width="0.1524" layer="91"/>
+<label x="40.64" y="78.74" size="1.27" layer="95" xref="yes"/>
+</segment>
+<segment>
+<pinref part="U3" gate="G$1" pin="SCL"/>
+<wire x1="40.64" y1="35.56" x2="43.18" y2="35.56" width="0.1524" layer="91"/>
+<label x="43.18" y="35.56" size="1.27" layer="95" xref="yes"/>
+</segment>
+<segment>
+<pinref part="U$7" gate="G$1" pin="SCLK"/>
+<wire x1="309.88" y1="208.28" x2="309.88" y2="195.58" width="0.1524" layer="91"/>
+<wire x1="309.88" y1="195.58" x2="304.8" y2="195.58" width="0.1524" layer="91"/>
+<label x="304.8" y="195.58" size="1.27" layer="95" rot="R180" xref="yes"/>
+</segment>
+</net>
+<net name="GPS_TX" class="0">
+<segment>
+<pinref part="U1" gate="G$1" pin="PA10(AIN18/SER0:2+)"/>
+<wire x1="200.66" y1="203.2" x2="203.2" y2="203.2" width="0.1524" layer="91" style="longdash"/>
+<label x="203.2" y="203.2" size="1.27" layer="95" xref="yes"/>
+</segment>
 <segment>
 <pinref part="U4" gate="G$1" pin="RX"/>

Commit message: lots of work on the layout
Parts:
- R10, R11, R12, R5, R6, R7, R8, R9: value (none) -> 10kohm; device SparkFun-Passives:RESISTOR0603-RES -> SparkFun-Resistors:RESISTOR0402
Connections:
- net FET_A: now also R9.2; no longer R9.1
- net FET_B: now also R11.1; no longer R11.2
- net FIRE_A: now also R5.2, R6.1, U1.PA19(SER1:3+); no longer R5.1, R6.2
- net FIRE_B: now also U1.PA21(SER5:3+)
- net GND: now also R10.1, R12.2, R5.1; no longer R10.2, R12.1, R6.1
- net N$1: now also R6.2; no longer R5.2
- net SENSE_A: now also R10.2, R9.1, U1.PA18(SER1:2+); no longer R10.1, R9.2
- net SENSE_B: now also R11.2, R12.1, U1.PA20(SER5:2+); no longer R11.1, R12.2
Other:
- moved on the sheet: R10, R11, R12, R5, R6, R9

Commit message: starting wiring
Parts:
- removed C16: (no value), SparkFun-Capacitors:CAP0402-CAP
- removed S1: SWITCH-MOMENTARY-2SMD-3, SparkFun-Electromechanical:SWITCH-MOMENTARY-2SMD-3
- added F1: PTCSMD, SparkFun-PowerIC:PTCSMD
- added S2: SWITCH-MOMENTARY-2SMD-4.6X2.8MM, SparkFun-Electromechanical:SWITCH-MOMENTARY-2SMD-4.6X2.8MM
- added SG1: BUZZERSMD2, SparkFun-Electromechanical:BUZZERSMD2
- added STANDOFF1, STANDOFF2, STANDOFF3: STAND-OFF, SparkFun-Electromechanical:STAND-OFF
- JP4: value USBSMD -> USB-MICROB; device SparkFun-Connectors:USBSMD -> SparkFun-Connectors:USB-MICROB
Connections:
- new net BUZZER: SG1.2, U1.PA18(SER1:2+)
- new net N$14: F1.1, JP4.VBUS
- new net SENSE_BAT: U1.PA04(AIN4/REFB/SER0:0/TC0:0)
- new net USB_D+: JP4.D+, U1.PA25(SER3:3+)
- new net USB_D-: JP4.D-, U1.PA24(SER3:2+)
- net 3.3V: now also S2.2; no longer S1.2
- net FIRE_A: now also U1.PA30(SWCLK/SER1:2+); no longer U1.PA19(SER1:3+)
- net FIRE_B: now also U1.PA31(SWDIO/SER1:3+); no longer U1.PA21(SER5:3+)
- net GND: now also JP4.GND, SG1.1
- net N$12: no longer C16.2
- net N$13: no longer C16.1
- net PROG: now also S2.1; no longer S1.1
- net SENSE_A: now also U1.PB08(AIN2/SER4:0/TC4:0); no longer U1.PA18(SER1:2+)
- net SENSE_B: now also U1.PB09(AIN3/SER4:1/TC4:1); no longer U1.PA20(SER5:2+)
- net SWCLK: no longer U1.PA30(SWCLK/SER1:2+)
- net SWDIO: no longer U1.PA31(SWDIO/SER1:3+)
Other:
- moved on the sheet: JP4

Commit message: more wiring
Connections:
- net CS_TX: now also U1.PA19(SER1:3+); no longer U1.PA16(I2C/SER1:0+)
- net GPS_RX: now also U1.PB23(SER5:3+); no longer U1.PA11(AIN19/SER0:3+)
- net GPS_TX: now also U1.PB22(SER5:2+); no longer U1.PA10(AIN18/SER0:2+)
- net PROG: now also U1.PA20(SER5:2+); no longer U1.PA17(I2C/SER1:1+)
- net SPI_MISO: now also U1.PA16(I2C/SER1:0+)
- net SPI_MOSI: now also U1.PA17(I2C/SER1:1+)
Changed lines of the file:
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@@
 </segment>
 <segment>
-<pinref part="U1" gate="G$1" pin="PA17(I2C/SER1:1+)"/>
-<wire x1="200.66" y1="185.42" x2="203.2" y2="185.42" width="0.1524" layer="91" style="longdash"/>
-<label x="203.2" y="185.42" size="1.27" layer="95" xref="yes"/>
+<pinref part="U1" gate="G$1" pin="PA20(SER5:2+)"/>
+<wire x1="200.66" y1="177.8" x2="203.2" y2="177.8" width="0.1524" layer="91"/>
+<label x="203.2" y="177.8" size="1.27" layer="95" xref="yes"/>
 </segment>
 </net>
@@
 </segment>
 <segment>
-<pinref part="U1" gate="G$1" pin="PA16(I2C/SER1:0+)"/>
-<wire x1="200.66" y1="187.96" x2="203.2" y2="187.96" width="0.1524" layer="91" style="longdash"/>
-<label x="203.2" y="187.96" size="1.27" layer="95" xref="yes"/>
+<pinref part="U1" gate="G$1" pin="PA19(SER1:3+)"/>
+<wire x1="200.66" y1="180.34" x2="203.2" y2="180.34" width="0.1524" layer="91"/>
+<label x="203.2" y="180.34" size="1.27" layer="95" xref="yes"/>
 </segment>
 </net>
@@
 </segment>
 <segment>
-<pinref part="U1" gate="G$1" pin="PA11(AIN19/SER0:3+)"/>
-<wire x1="200.66" y1="200.66" x2="203.2" y2="200.66" width="0.1524" layer="91" style="longdash"/>
-<label x="203.2" y="200.66" size="1.27" layer="95" xref="yes"/>
+<pinref part="U1" gate="G$1" pin="PB23(SER5:3+)"/>
+<wire x1="200.66" y1="142.24" x2="203.2" y2="142.24" width="0.1524" layer="91"/>
+<label x="203.2" y="142.24" size="1.27" layer="95" xref="yes"/>
 </segment>
 </net>
@@
 <wire x1="320.04" y1="193.04" x2="304.8" y2="193.04" width="0.1524" layer="91"/>
 <label x="304.8" y="193.04" size="1.27" layer="95" rot="R180" xref="yes"/>
+</segment>
+<segment>
+<pinref part="U1" gate="G$1" pin="PA16(I2C/SER1:0+)"/>
+<wire x1="200.66" y1="187.96" x2="203.2" y2="187.96" width="0.1524" layer="91" style="longdash"/>
+<label x="203.2" y="187.96" size="1.27" layer="95" xref="yes"/>
 </segment>
 </net>
@@
 <label x="304.8" y="198.12" size="1.27" layer="95" rot="R180" xref="yes"/>
 </segment>
+<segment>
+<pinref part="U1" gate="G$1" pin="PA17(I2C/SER1:1+)"/>
+<wire x1="200.66" y1="185.42" x2="203.2" y2="185.42" width="0.1524" layer="91" style="longdash"/>
+<label x="203.2" y="185.42" size="1.27" layer="95" xref="yes"/>
+</segment>
 </net>
 <net name="SPI_SCK" class="0">
@@
 <net name="GPS_TX" class="0">
 <segment>
-<pinref part="U1" gate="G$1" pin="PA10(AIN18/SER0:2+)"/>
-<wire x1="200.66" y1="203.2" x2="203.2" y2="203.2" width="0.1524" layer="91" style="longdash"/>
-<label x="203.2" y="203.2" size="1.27" layer="95" xref="yes"/>
-</segment>
-<segment>
 <pinref part="U4" gate="G$1" pin="RX"/>
 <wire x1="340.36" y1="86.36" x2="337.82" y2="86.36" width="0.1524" layer="91"/>
 <label x="337.82" y="86.36" size="1.27" layer="95" rot="R180" xref="yes"/>
 </segment>
-</net>
+<segment>
+<pinref part="U1" gate="G$1" pin="PB22(SER5:2+)"/>
+<wire x1="200.66" y1="144.78" x2="203.2" y2="144.78" width="0.1524" layer="91"/>
+<label x="203.2" y="144.78" size="1.27" layer="95" xref="yes"/>
+</segment>
+</net>

Commit message: finshed wiring
Parts:
- added R18: 100k, SparkFun-Passives:RESISTOR0402-RES
- added R19: 27k, SparkFun-Passives:RESISTOR0402-RES
- added R20: 10k, SparkFun-Passives:RESISTOR0402-RES
- C8: value (none) -> 0.1uF
- J1: value (none) -> BAT
- JP2: value (none) -> MAIN
- JP3: value (none) -> DROGUE
- R1, R13, R2, R3, R4: value (none) -> 10k
- R15: value (none) -> 18
- U4: value (none) -> gps
- Y1: value (none) -> 32.768kHx
Connections:
- removed net N$7: U1.VDDANA
- net BUZZER: now also SG1.1, U1.PA12(I2C/SER2:0+); no longer SG1.2, U1.PA18(SER1:2+)
- net CS_ACCEL: now also U1.PA16(I2C/SER1:0+); no longer U1.PA15(XOUT/SER2:3+)
- net CS_BARO: now also U1.PA09(I2C/AIN17/SER0:1+); no longer U1.PA13(I2C/SER2:1+)
- net CS_MEM: now also U1.PA08(I2C/AIN16/SER0:0+); no longer U1.PA14(XIN/SER2:2+)
- net CS_TX: now also R20.1, U1.PA10(AIN18/SER0:2+); no longer U1.PA19(SER1:3+)
- net FIRE_A: now also U1.PB02(AIN10/SER5:0); no longer U1.PA30(SWCLK/SER1:2+)
- net FIRE_B: now also U1.PB03(AIN11/SER5:1); no longer U1.PA31(SWDIO/SER1:3+)
- net GND: now also R19.1, R20.2, SG1.2, U$7.EP; no longer SG1.1
- net LVD_IN: now also F1.2
- net N$5: now also U1.VDDANA
- net PROG: now also U1.PA07(AIN7/SER0:3/TC1:1); no longer U1.PA20(SER5:2+)
- net RAW: now also R18.2
- net SENSE_BAT: now also R18.1, R19.2, U1.PA06(AIN6/SER0:2/TC1:0); no longer U1.PA04(AIN4/REFB/SER0:0/TC0:0)
- net SPI_MISO: now also U1.PA14(XIN/SER2:2+); no longer U1.PA12(I2C/SER2:0+), U1.PA16(I2C/SER1:0+)
- net SPI_MOSI: now also U1.PA13(I2C/SER2:1+); no longer U1.PA17(I2C/SER1:1+), U1.PB10(SER4:2+)
- net SPI_SCK: now also U1.PA15(XOUT/SER2:3+); no longer U1.PB11(SER4:3+)
- net SWCLK: now also U1.PA30(SWCLK/SER1:2+)
- net SWDIO: now also U1.PA31(SWDIO/SER1:3+)

Commit message: mk1 finished!
Parts:
- removed U$7: CC1120, SaL-lib:CC1120
- added 1U2: V_REG_LDOSMD, SparkFun-PowerIC:V_REG_LDOSMD
- U2: value V_REG_LDOSMD -> CC1120; device SparkFun-PowerIC:V_REG_LDOSMD -> SaL-lib:CC1120
- renumbered U$4 to MEM
Connections:
- net 3.3V: now also 1U2.OUT, U2.AVDD_IF, U2.AVDD_RF, U2.AVDD_SYNTH1, U2.AVDD_SYNTH2, U2.AVDD_XOSC, U2.DVDD, U2.DVDD1, U2.VDD_GUARD; no longer U$7.AVDD_IF, U$7.AVDD_RF, U$7.AVDD_SYNTH1, U$7.AVDD_SYNTH2, U$7.AVDD_XOSC, U$7.DVDD, U$7.DVDD1, U$7.VDD_GUARD, U2.OUT
- net CS_TX: now also U2.CSN; no longer U$7.CSN
- net FET_A: now also JP2.2; no longer JP2.1
- net GND: now also 1U2.GND, U2.EP; no longer U$7.EP, U2.GND
- net LVD_IN: now also 1U2.EN, 1U2.IN, JP2.1; no longer JP2.2, U2.EN, U2.IN
- net N$15: now also U2.AVDD_PFD_CHP; no longer U$7.AVDD_PFD_CHP
- net N$16: now also U2.TRX_SW; no longer U$7.TRX_SW
- net N$17: now also U2.LNA_P; no longer U$7.LNA_P
- net N$19: now also U2.LNA_N; no longer U$7.LNA_N
- net N$20: now also U2.LPF1; no longer U$7.LPF1
- net N$21: now also U2.LPF0; no longer U$7.LPF0
- net N$22: now also U2.DCPL_VCO; no longer U$7.DCPL_VCO
- net N$23: now also U2.DCPL_PFD_CHP; no longer U$7.DCPL_PFD_CHP
- net N$24: now also U2.RBIAS; no longer U$7.RBIAS
- net N$25: now also U2.EXT_XOSC; no longer U$7.EXT_XOSC
- net N$26: now also U2.DCPL_XOSC; no longer U$7.DCPL_XOSC
- net N$27: now also U2.XOSC_Q1; no longer U$7.XOSC_Q1
- net N$28: now also U2.XOSC_Q2; no longer U$7.XOSC_Q2
- net N$34: now also U2.DCPL; no longer U$7.DCPL
- net N$9: now also U2.PA; no longer U$7.PA
- net SPI_MISO: now also U2.GPOI1; no longer U$7.GPOI1
- net SPI_MOSI: now also U2.SI; no longer U$7.SI
- net SPI_SCK: now also U2.SCLK; no longer U$7.SCLK

Commit message: parts lists added
Parts:
- C1: value 1.0uF -> 2.2uF
- R10, R12: value 10kohm -> 27K
- R11, R9: value 10kohm -> 100K
- R5, R8: value 10kohm -> 3.3k
- R6, R7: value 10kohm -> 100
Changed lines of the file:
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@@
 <part name="SUPPLY1" library="SparkFun-Aesthetics" deviceset="3.3V" device=""/>
 <part name="GND1" library="SparkFun-Aesthetics" deviceset="GND" device=""/>
-<part name="C1" library="SparkFun-Capacitors" deviceset="CAP" device="0603-CAP" value="1.0uF"/>
+<part name="C1" library="SparkFun-Capacitors" deviceset="CAP" device="0603-CAP" value="2.2uF"/>
 <part name="C2" library="SparkFun-Capacitors" deviceset="CAP" device="0603-CAP" value="2.2uF"/>
 <part name="U$1" library="SaL-lib" deviceset="MAX16054" device=""/>
@@
 <part name="SUPPLY22" library="SparkFun-Aesthetics" deviceset="3.3V" device=""/>
 <part name="GND46" library="SparkFun-Aesthetics" deviceset="GND" device=""/>
-<part name="R5" library="SparkFun-Resistors" deviceset="RESISTOR" device="0402" value="10kohm"/>
-<part name="R6" library="SparkFun-Resistors" deviceset="RESISTOR" device="0402" value="10kohm"/>
-<part name="R9" library="SparkFun-Resistors" deviceset="RESISTOR" device="0402" value="10kohm"/>
-<part name="R10" library="SparkFun-Resistors" deviceset="RESISTOR" device="0402" value="10kohm"/>
-<part name="R7" library="SparkFun-Resistors" deviceset="RESISTOR" device="0402" value="10kohm"/>
-<part name="R8" library="SparkFun-Resistors" deviceset="RESISTOR" device="0402" value="10kohm"/>
-<part name="R11" library="SparkFun-Resistors" deviceset="RESISTOR" device="0402" value="10kohm"/>
-<part name="R12" library="SparkFun-Resistors" deviceset="RESISTOR" device="0402" value="10kohm"/>
+<part name="R5" library="SparkFun-Resistors" deviceset="RESISTOR" device="0402" value="3.3k"/>
+<part name="R6" library="SparkFun-Resistors" deviceset="RESISTOR" device="0402" value="100"/>
+<part name="R9" library="SparkFun-Resistors" deviceset="RESISTOR" device="0402" value="100K"/>
+<part name="R10" library="SparkFun-Resistors" deviceset="RESISTOR" device="0402" value="27K"/>
+<part name="R7" library="SparkFun-Resistors" deviceset="RESISTOR" device="0402" value="100"/>
+<part name="R8" library="SparkFun-Resistors" deviceset="RESISTOR" device="0402" value="3.3k"/>
+<part name="R11" library="SparkFun-Resistors" deviceset="RESISTOR" device="0402" value="100K"/>
+<part name="R12" library="SparkFun-Resistors" deviceset="RESISTOR" device="0402" value="27K"/>
 <part name="JP4" library="SparkFun-Connectors" deviceset="USB" device="-MICROB"/>
 <part name="F1" library="SparkFun-PowerIC" deviceset="PTC" device="SMD"/>
